File: AIR.sch (EAGLE design)
At the start: 32 parts

Commit message: Updated EAGLE files
Parts:
- CE1, CE2, CE3, CE4: value 100uF -> 100µF
Changed lines of the file:
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@@
 <part name="C1" library="rcl" deviceset="C-EU" device="025-025X050" value="0.1µF"/>
 <part name="C2" library="rcl" deviceset="C-EU" device="025-025X050" value="0.1µF"/>
-<part name="CE1" library="Eagle_Wurth_Elektronik_Passive_Capacitors_rev15a" deviceset="WCAP-PTG5" device="_8X8X3.5X0.6(DXLXPXØ)" value="100uF"/>
-<part name="CE2" library="Eagle_Wurth_Elektronik_Passive_Capacitors_rev15a" deviceset="WCAP-PTG5" device="_8X8X3.5X0.6(DXLXPXØ)" value="100uF"/>
+<part name="CE1" library="Eagle_Wurth_Elektronik_Passive_Capacitors_rev15a" deviceset="WCAP-PTG5" device="_8X8X3.5X0.6(DXLXPXØ)" value="100µF"/>
+<part name="CE2" library="Eagle_Wurth_Elektronik_Passive_Capacitors_rev15a" deviceset="WCAP-PTG5" device="_8X8X3.5X0.6(DXLXPXØ)" value="100µF"/>
 <part name="C5" library="rcl" deviceset="C-EU" device="025-025X050" value="0.1µF"/>
 <part name="L293D2/1" library="Wurth_Elektronik_Electromechanic_Board_to_Board_Connectors_rev15b" deviceset="61300811821" device=""/>
@@
 <part name="C6" library="rcl" deviceset="C-EU" device="025-025X050" value="0.1µF"/>
 <part name="C7" library="rcl" deviceset="C-EU" device="025-025X050" value="0.1µF"/>
-<part name="CE3" library="Eagle_Wurth_Elektronik_Passive_Capacitors_rev15a" deviceset="WCAP-PTG5" device="_8X8X3.5X0.6(DXLXPXØ)" value="100uF"/>
-<part name="CE4" library="Eagle_Wurth_Elektronik_Passive_Capacitors_rev15a" deviceset="WCAP-PTG5" device="_8X8X3.5X0.6(DXLXPXØ)" value="100uF"/>
+<part name="CE3" library="Eagle_Wurth_Elektronik_Passive_Capacitors_rev15a" deviceset="WCAP-PTG5" device="_8X8X3.5X0.6(DXLXPXØ)" value="100µF"/>
+<part name="CE4" library="Eagle_Wurth_Elektronik_Passive_Capacitors_rev15a" deviceset="WCAP-PTG5" device="_8X8X3.5X0.6(DXLXPXØ)" value="100µF"/>
 <part name="C10" library="rcl" deviceset="C-EU" device="025-025X050" value="0.1µF"/>
 <part name="GND8" library="supply1" deviceset="GND" device=""/>

Commit message: Major improvements on hardware, patch stability
Parts:
- removed MAINS/BATT, MOT/B, MOT/C, MOT/L, MOT/R: 691101710002, Wurth_Elektronik_Electromechanic_Terminal_Blocks_Connectors_rev15b:691101710002
- added BATT/CHRG: 691121710004, Wurth_Elektronik_Electromechanic_Terminal_Blocks_Connectors_rev15b:691121710004
- added MOTORS/BLCR: 691221320008, Wurth_Elektronik_Electromechanic_Terminal_Blocks_Connectors_rev15b:691221320008
- MAINS/SW: value 691101710002 -> 691101710003; device Wurth_Elektronik_Electromechanic_Terminal_Blocks_Connectors_rev15b:691101710002 -> Wurth_Elektronik_Electromechanic_Terminal_Blocks_Connectors_rev15b:691101710003
Connections:
- new net N$4: BATT/CHRG.4, MAINS/SW.3
- net +24V: now also MAINS/SW.1; no longer MAINS/SW.2
- net GND: now also BATT/CHRG.2, BATT/CHRG.3; no longer MAINS/BATT.2
- net MB+: now also MOTORS/BLCR.1; no longer MOT/B.1
- net MB-: now also MOTORS/BLCR.2; no longer MOT/B.2
- net MC+: now also MOTORS/BLCR.5; no longer MOT/C.1
- net MC-: now also MOTORS/BLCR.6; no longer MOT/C.2
- net ML+: now also MOTORS/BLCR.3; no longer MOT/L.1
- net ML-: now also MOTORS/BLCR.4; no longer MOT/L.2
- net MR+: now also MOTORS/BLCR.7; no longer MOT/R.1
- net MR-: now also MOTORS/BLCR.8; no longer MOT/R.2
- net N$3: now also BATT/CHRG.1, MAINS/SW.2; no longer MAINS/BATT.1, MAINS/SW.1
Other:
- moved on the sheet: DCDCCONV
